File: HARDWARE/AquarWorld - Circuito/AquarWorld - Circuito.kicad_pcb (KiCad board)
At the start: 2 copper layers, 147.7 x 90.8 mm, 69 parts, among them J10 SALIDA - RELAY 1, J13 12V - GND, J15 5V - GND, J2 MP3-PLAYER, J27 ALIMENTACIÓN - 12V, J4 SALIDA - RELAY 2, J5 SENSOR ULTRASONICO, J6 SALIDA - RELAY 3, J7 SALIDA - RELAY 4, K1 RELAY 2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

Commit message: Placa principal - AquarWorld
Connections:
- R39 pad 1: ECHO -> Net-(J5-Pin_3)
- R39 pad 2: Net-(J5-Pin_3) -> ECHO
- R40 pad 1: Net-(J5-Pin_3) -> ECHO
- U2 pad 12: TRIG -> unconnected-(U2-IO14-Pad12)
- U2 pad 15: ECHO -> unconnected-(U2-IO13-Pad15)
- U2 pad 24: RELAY 4 -> unconnected-(U2-IO2-Pad24)
- U2 pad 26: RELAY 3 -> unconnected-(U2-IO4-Pad26)
- U2 pad 28: RELAY 2 -> RELAY 4
- U2 pad 30: RELAY 1 -> RELAY 3
- U2 pad 36: unconnected-(U2-IO22-Pad36) -> RELAY 2
- U2 pad 37: unconnected-(U2-IO23-Pad37) -> RELAY 1
- U2 pad 6: unconnected-(U2-IO35-Pad6) -> TRIG
- U2 pad 7: unconnected-(U2-IO32-Pad7) -> ECHO
Routing:
- net ECHO: track 65.1 -> 45.0 mm, vias 1 -> 0
- net RELAY 1: track 45.7 -> 28.5 mm
- net TRIG: track 60.4 -> 45.6 mm
- net RELAY 3: track 17.0 -> 26.5 mm
- net RELAY 2: track 30.3 -> 21.1 mm
- net RELAY 4: track 32.9 -> 41.9 mm
- net Net-(J5-Pin_3): track 21.6 -> 12.8 mm
- net unconnected-(U2-IO14-Pad12): track 0.00 -> 3.99 mm
