File: HARDWARE/AquarWorld - Circuito/AquarWorld - Circuito.kicad_sch (KiCad schematic)
At the start: 80 parts, among them J10 SALIDA - RELAY 1, J13 12V - GND, J15 5V - GND, J2 MP3-PLAYER, J27 ALIMENTACIÓN - 12V, J3 SENSOR DE TEMPERATURA, J4 SALIDA - RELAY 2, J5 SENSOR ULTRASONICO, J6 SALIDA - RELAY 3, J7 SALIDA - RELAY 4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

Commit message: Placa pricipal - AquarWorld
Parts:
- removed D12, D13: LED, Connector_JST:JST_XH_B2B-XH-A_1x02_P2.50mm_Vertical, symbol Device:LED
- removed J3: SENSOR DE TEMPERATURA, Connector_JST:JST_XH_B3B-XH-A_1x03_P2.50mm_Vertical, symbol Connector:Conn_01x03_Pin
- removed R19, R22, R25: 1KΩ, Resistor_SMD:R_0805_2012Metric, symbol Device:R_US
- removed R30, R31: 220Ω, Resistor_SMD:R_0805_2012Metric, symbol Device:R_US
- removed SW1: PULSADOR 1, Connector_JST:JST_XH_B2B-XH-A_1x02_P2.50mm_Vertical, symbol Switch:SW_Push
- removed SW4: PULSADOR 2, Connector_JST:JST_XH_B2B-XH-A_1x02_P2.50mm_Vertical, symbol Switch:SW_Push
- removed SW7: PULSADOR 3, Connector_JST:JST_XH_B2B-XH-A_1x02_P2.50mm_Vertical, symbol Switch:SW_Push
Connections:
- net PULSADOR 1 is gone; now on net ECHO: U2.15 (IO13)
- net PULSADOR 2 is gone; now on net TRIG: U2.12 (IO14)
- net BUZZER: now also U2.33 (IO21); no longer U2.23 (IO15)
- net ECHO: no longer U2.10 (IO26)
- net TRIG: no longer U2.9 (IO25)
- net LED - ADVERTENCIA 3: no longer names the net of U2.6 (IO35)
- net LED - ADVERTENCIA 4: no longer names the net of U2.5 (IO34)
- net PULSADOR 3: no longer names the net of U2.11 (IO27)
- net SENSOR DE TEMPERATURA: no longer names the net of U2.7 (IO32)
- no-connect marks 14 -> 20
Other:
- note removed: "ETAPA N°5: PULSADORES - OPCIONES"
- moved on the sheet: D10, D11, R28, R29
