File: HARDWARE/AquarWorld - Circuito/AquarWorld - Circuito.kicad_sch (KiCad schematic)
At the start: 69 parts, among them J10 SALIDA - RELAY 1, J13 12V - GND, J15 5V - GND, J2 MP3-PLAYER, J27 ALIMENTACIÓN - 12V, J4 SALIDA - RELAY 2, J5 SENSOR ULTRASONICO, J6 SALIDA - RELAY 3, J7 SALIDA - RELAY 4, K1 RELAY 2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

Commit message: Placa principal - AquarWorld
Connections:
- net ECHO: now also R39.2, R40.1, U2.7 (IO32); no longer R39.1, U2.15 (IO13)
- net RELAY 1: now also U2.37 (IO23); no longer U2.30 (IO18)
- net RELAY 2: now also U2.36 (IO22); no longer U2.28 (IO17)
- net RELAY 3: now also U2.30 (IO18); no longer U2.26 (IO4)
- net RELAY 4: now also U2.28 (IO17); no longer U2.24 (IO2)
- net TRIG: now also U2.6 (IO35); no longer U2.12 (IO14)
- new net: J5.3 (Pin_3), R39.1
- no-connect marks 20 -> 21
Changed lines of the file:
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@@
 	)
 	(junction
+		(at 332.74 335.28)
+		(diameter 0)
+		(color 0 0 0 0)
+	)
+	(junction
 		(at 581.66 247.65)
 		(diameter 0)
@@
 	)
 	(junction
-		(at 332.74 335.28)
-		(diameter 0)
-		(color 0 0 0 0)
-	)
-	(junction
 		(at 204.47 177.8)
 		(diameter 0)
@@
 	)
 	(no_connect
+		(at 171.45 337.82)
+	)
+	(no_connect
 		(at 130.81 345.44)
 	)
@@
 	)
 	(no_connect
-		(at 130.81 304.8)
+		(at 171.45 332.74)
 	)
 	(no_connect
-		(at 130.81 322.58)
+		(at 130.81 304.8)
 	)
 	(no_connect
-		(at 130.81 327.66)
+		(at 130.81 330.2)
 	)
 	(no_connect
-		(at 171.45 307.34)
+		(at 130.81 322.58)
 	)
 	(no_connect
-		(at 171.45 304.8)
+		(at 130.81 327.66)
 	)
 	(no_connect
@@
 	)
 	(no_connect
-		(at 130.81 314.96)
-	)
-	(no_connect
 		(at 171.45 345.44)
 	)
@@
 	)
 	(no_connect
+		(at 130.81 337.82)
+	)
+	(no_connect
 		(at 171.45 320.04)
 	)
@@
 	(wire
 		(pts
-			(xy 332.74 334.01) (xy 332.74 335.28)
+			(xy 332.74 344.17) (xy 332.74 346.71)
 		)
 		(stroke
@@
 	(wire
 		(pts
+			(xy 341.63 322.58) (xy 332.74 322.58)
+		)
+		(stroke
+			(width 0)
+			(type default)
+		)
+	)
+	(wire
+		(pts
 			(xy 317.5 129.54) (xy 321.31 129.54)
 		)
@@
 	(wire
 		(pts
+			(xy 332.74 322.58) (xy 332.74 326.39)
+		)
+		(stroke
+			(width 0)
+			(type default)
+		)
+	)
+	(wire
+		(pts
 			(xy 125.73 347.98) (xy 130.81 347.98)
 		)
@@
 	(wire
 		(pts
+			(xy 332.74 335.28) (xy 332.74 336.55)
+		)
+		(stroke
+			(width 0)
+			(type default)
+		)
+	)
+	(wire
+		(pts
 			(xy 173.99 200.66) (xy 173.99 205.74)
 		)
@@
 	(wire
 		(pts
-			(xy 332.74 335.28) (xy 332.74 336.55)
+			(xy 332.74 334.01) (xy 332.74 335.28)
 		)
 		(stroke
@@
 	(wire
 		(pts
+			(xy 326.39 335.28) (xy 332.74 335.28)
+		)
+		(stroke
+			(width 0)
+			(type default)
+		)
+	)
+	(wire
+		(pts
 			(xy 557.53 229.87) (xy 557.53 223.52)
 		)
@@
 	(wire
 		(pts
+			(xy 341.63 335.28) (xy 341.63 322.58)
+		)
+		(stroke
+			(width 0)
+			(type default)
+		)
+	)
+	(wire
+		(pts
 			(xy 171.45 302.26) (xy 191.77 302.26)
 		)
@@
 	(wire
 		(pts
+			(xy 341.63 335.28) (xy 356.87 335.28)
+		)
+		(stroke
+			(width 0)
+			(type default)
+		)
+	)
+	(wire
+		(pts
 			(xy 317.5 240.03) (xy 317.5 234.95)
 		)
@@
 	(wire
 		(pts
-			(xy 332.74 335.28) (xy 356.87 335.28)
-		)
-		(stroke
-			(width 0)
-			(type default)
-		)
-	)
-	(wire
-		(pts
 			(xy 389.89 201.93) (xy 407.67 201.93)
 		)
@@
 	(global_label "ECHO"
 		(shape input)
-		(at 130.81 337.82 180)
+		(at 130.81 317.5 180)
 		(fields_autoplaced yes)
 		(effects
@@
 		)
 		(property "Intersheetrefs" "${INTERSHEET_REFS}"
-			(at 122.7448 337.82 0)
+			(at 122.7448 317.5 0)
 			(effects
 				(font
@@
 	(global_label "RELAY 2"
 		(shape input)
-		(at 171.45 327.66 0)
+		(at 171.45 307.34 0)
 		(fields_autoplaced yes)
 		(effects
@@
 		)
 		(property "Intersheetrefs" "${INTERSHEET_REFS}"
-			(at 182.2366 327.66 0)
+			(at 182.2366 307.34 0)
 			(effects
 				(font
@@
 	(global_label "RELAY 4"
 		(shape input)
-		(at 171.45 337.82 0)
+		(at 171.45 327.66 0)
 		(fields_autoplaced yes)
 		(effects
@@
 		)
 		(property "Intersheetrefs" "${INTERSHEET_REFS}"
-			(at 182.2366 337.82 0)
+			(at 182.2366 327.66 0)
 			(effects
 				(font
@@
 	(global_label "RELAY 3"
 		(shape input)
-		(at 171.45 332.74 0)
+		(at 171.45 322.58 0)
 		(fields_autoplaced yes)
 		(effects
@@
 		)
 		(property "Intersheetrefs" "${INTERSHEET_REFS}"
-			(at 182.2366 332.74 0)
+			(at 182.2366 322.58 0)
 			(effects
 				(font
@@
 	(global_label "RELAY 1"
 		(shape input)
-		(at 171.45 322.58 0)
+		(at 171.45 304.8 0)
 		(fields_autoplaced yes)
 		(effects
@@
 		)
 		(property "Intersheetrefs" "${INTERSHEET_REFS}"
-			(at 182.2366 322.58 0)
+			(at 182.2366 304.8 0)
 			(effects
 				(font
@@
 	(global_label "TRIG"
 		(shape input)
-		(at 130.81 330.2 180)
+		(at 130.81 314.96 180)
 		(fields_autoplaced yes)
 		(effects
@@
 		)
 		(property "Intersheetrefs" "${INTERSHEET_REFS}"
-			(at 123.7124 330.2 0)
+			(at 123.7124 314.96 0)
 			(effects
 				(font
@@
 	(global_label "ECHO"
 		(shape input)
-		(at 332.74 326.39 90)
+		(at 326.39 335.28 180)
 		(fields_autoplaced yes)
 		(effects
@@
 				(size 1.27 1.27)
 			)
-			(justify left)
+			(justify right)
 		)
 		(property "Intersheetrefs" "${INTERSHEET_REFS}"
-			(at 332.74 318.3248 90)
+			(at 318.3248 335.28 0)
 			(effects
 				(font
 					(size 1.27 1.27)
 				)
-				(justify left)
+				(justify right)
 				(hide yes)
 			)
@@
 		(lib_name "Earth_1")
 		(lib_id "power:Earth")
-		(at 332.74 344.17 0)
+		(at 332.74 346.71 0)
 		(unit 1)
 		(exclude_from_sim no)
@@
 		(dnp no)
 		(property "Reference" "#PWR055"
-			(at 332.74 350.52 0)
+			(at 332.74 353.06 0)
 			(effects
 				(font
@@
 		)
 		(property "Value" "Earth"
-			(at 332.74 347.98 0)
+			(at 332.74 350.52 0)
 			(effects
 				(font
@@
 		)
 		(property "Footprint" ""
-			(at 332.74 344.17 0)
+			(at 332.74 346.71 0)
 			(effects
 				(font
@@
 		)
 		(property "Datasheet" "~"
-			(at 332.74 344.17 0)
+			(at 332.74 346.71 0)
 			(effects
 				(font
@@
 		)
 		(property "Description" ""
-			(at 332.74 344.17 0)
+			(at 332.74 346.71 0)
 			(effects
 				(font
