File: HARDWARE/Lanzador de pelotas - Iván Barrientos - ELECTRÓNICA 2025/Lanzador de pelotas - Iván Barrientos - ELECTRÓNICA 2025.kicad_pcb (KiCad board)
At the start: 2 copper layers, 63.6 x 54 mm, 21 parts, among them J1 ALIMENTACIÓN-12V, J2 12V, J5 SENSOR IFLAROJO (IR), J6 APAGADO/ENCENDIDO, J7 PUENTE H - L298N, Q1 2N7000, U1 ESP32-C3_SUPERMINI, U2 L7805

Commit message: Lanzador de pelotas - Iván Barrientos
Parts:
- added D5: 1N4007, Diode_THT:D_A-405_P10.16mm_Horizontal, F.Cu at (134.1, 91.5)
- moved U2 3.84 mm to (125.5, 80.2)
- moved JP1 3.77 mm to (123.5, 91.1)
- moved J2 3.77 mm to (127.8, 93.7)
- moved J6 3.77 mm to (124.4, 99.9)
- moved C1 2.46 mm to (118.3, 115.9)
- moved C2 2.46 mm to (130.1, 115.9)
- moved D1 2.46 mm to (115.9, 82.3)
- moved R1 2.46 mm to (115.9, 79.8)
- moved J1 2.20 mm to (115.0, 99.5)
Connections:
- D2 pad 1: Earth -> LED 1 - 30CM
- D3 pad 1: Earth -> LED 2 - 60CM
- D4 pad 1: Earth -> LED 3 - 90CM
- R3 pad 2: LED 1 - 30CM -> +3.3V
- R4 pad 2: LED 2 - 60CM -> +3.3V
- R5 pad 2: LED 3 - 90CM -> +3.3V
- U1 pad 0: LED 1 - 30CM -> ENB - B
- U1 pad 2: ENB - B -> LED 1 - 30CM
- U1 pad 3: LED 2 - 60CM -> +3.3V
- U1 pad 3.3: unconnected-(U1-3V3-Pad3.3) -> +3.3V
- U1 pad 5V: +5V -> Net-(D5-K)
Routing:
- net +3.3V: track 0.00 -> 80.2 mm, vias 0 -> 2
- net +5V: track 124.0 -> 153.9 mm, vias 2 -> 1
- net LED 1 - 30CM: track 11.3 -> 24.3 mm, vias 1 -> 0
- net LED 2 - 60CM: track 9.49 -> 0.00 mm, vias 1 -> 0
- net Net-(D5-K): track 0.00 -> 7.51 mm
- net LED 3 - 90CM: track 11.5 -> 14.5 mm, vias 1 -> 0
- net ENB - B: track 20.1 -> 22.9 mm
- net +12V: track 69.9 -> 69.2 mm
Other:
- board size 63.6 x 54 mm -> 66.3 x 54 mm

Commit message: Lanzador de pelotas
Parts:
- D5: footprint Diode_THT:D_A-405_P10.16mm_Horizontal -> Diode_SMD:D_0805_2012Metric
- moved D5 5.01 mm to (134.7, 96.5)
- moved C1 2.20 mm to (120.5, 115.9)
- moved J6 2.20 mm to (126.6, 99.9)
- moved JP1 2.20 mm to (125.7, 91.1)
- moved R1 2.20 mm to (118.1, 79.8)
- moved U2 2.20 mm to (127.7, 80.2)
- moved C2 2.20 mm to (132.3, 115.9)
- moved D1 2.20 mm to (118.1, 82.3)
- moved J1 2.20 mm to (117.2, 99.5)
- moved J2 2.20 mm to (130.0, 93.7)
Connections:
- U1 pad 3: +3.3V -> LED 2 - 60CM
Routing:
- net +5V: track 153.9 -> 116.3 mm
- net Net-(D5-K): track 7.51 -> 11.8 mm, vias 0 -> 1
Other:
- board size 66.3 x 54 mm -> 63.7 x 54 mm
