File: HARDWARE/Lanzador de pelotas - Iván Barrientos - ELECTRÓNICA 2025/Lanzador de pelotas - Iván Barrientos - ELECTRÓNICA 2025.kicad_sch (KiCad schematic)
At the start: 21 parts, among them J1 ALIMENTACIÓN-12V, J2 12V, J5 SENSOR IFLAROJO (IR), J6 APAGADO/ENCENDIDO, J7 PUENTE H - L298N, Q1 2N7000, U1 ESP32-C3_SUPERMINI, U2 L7805

Commit message: Lanzador de pelotas - Iván Barrientos
Parts:
- added D5: 1N4007, Diode_THT:D_A-405_P10.16mm_Horizontal, symbol Device:D
Connections:
- net +5V: now also D5.2 (A); no longer U1.5V
- net ENB - B: now also U1.0 (GPIO0); no longer U1.2 (GPIO2)
- net Earth: no longer D2.1 (K), D3.1 (K), D4.1 (K)
- net LED 1 - 30CM: now also D2.1 (K), U1.2 (GPIO2); no longer R3.2, U1.0 (GPIO0)
- net LED 2 - 60CM: now also D3.1 (K); no longer R4.2
- net LED 3 - 90CM: now also D4.1 (K); no longer R5.2
- net +3.3V: now reaches U1.3.3 (3V3)
- net +3.3V: now also R3.2, R4.2, R5.2
- new net: D5.1 (K), U1.5V
- no-connect marks 3 -> 2

Commit message: Lanzador de pelotas
Parts:
- D5: footprint Diode_THT:D_A-405_P10.16mm_Horizontal -> Diode_SMD:D_0805_2012Metric
Changed lines of the file:
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@@
 			)
 		)
-		(property "Footprint" "Diode_THT:D_A-405_P10.16mm_Horizontal"
+		(property "Footprint" "Diode_SMD:D_0805_2012Metric"
 			(at 111.76 186.69 0)
 			(effects
